File: elec/layout/default/mmmm-whats-your-name.kicad_pcb (KiCad board)
At the start: 2 copper layers, 225.7 x 100.8 mm, 0 parts

Commit message: Rough blocks are in the right places
Parts:
- added C1: Multilayer Ceramic Capacitors MLCC - SMD/SMT 10uF 10V 0805 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, lib:C0805, F.Cu at (134.1, 46.2)
- added C10: Multilayer Ceramic Capacitors MLCC - SMD/SMT 100nF 10V 0402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, lib:C0402, F.Cu at (141.6, 59.1)
- added C11: Multilayer Ceramic Capacitors MLCC - SMD/SMT 1uF 6.3V 0402 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, lib:C0402, F.Cu at (144.4, 46.4)
- added C12: Multilayer Ceramic Capacitors MLCC - SMD/SMT 1uF 6.3V 0402 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, lib:C0402, F.Cu at (144.4, 42.9)
- added C13: Multilayer Ceramic Capacitors MLCC - SMD/SMT 20pF 50V 0402 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, lib:C0402, F.Cu at (118.1, 63.4)
- added C14: Multilayer Ceramic Capacitors MLCC - SMD/SMT 20pF 50V 0402 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, lib:C0402, F.Cu at (123.4, 64.2)
- added C15: Multilayer Ceramic Capacitors MLCC - SMD/SMT 100nF 10V 0402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, lib:C0402, F.Cu at (123.5, 62.3)
- added C16: Multilayer Ceramic Capacitors MLCC - SMD/SMT 100nF 10V 0402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, lib:C0402, F.Cu at (127.5, 52.5)
- added C17: Multilayer Ceramic Capacitors MLCC - SMD/SMT 100nF 10V 0402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, lib:C0402, F.Cu at (116.9, 51.4)
- added C18: Multilayer Ceramic Capacitors MLCC - SMD/SMT 100nF 10V 0402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, lib:C0402, F.Cu at (116.9, 52.5)
- added C19: Multilayer Ceramic Capacitors MLCC - SMD/SMT 100nF 10V 0402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, lib:C0402, F.Cu at (127.6, 56.3)
- added C2: Multilayer Ceramic Capacitors MLCC - SMD/SMT 10uF 10V 0805 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, lib:C0805, F.Cu at (134.1, 44.2)
- added C20: Multilayer Ceramic Capacitors MLCC - SMD/SMT 1uF 6.3V 0402 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, lib:C0402, F.Cu at (125.8, 43.2)
- added C21: Multilayer Ceramic Capacitors MLCC - SMD/SMT 100nF 10V 0402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, lib:C0402, F.Cu at (122.1, 50.0)
- added C22: Multilayer Ceramic Capacitors MLCC - SMD/SMT 100nF 10V 0402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, lib:C0402, F.Cu at (127.5, 51.4)
- added C23: Multilayer Ceramic Capacitors MLCC - SMD/SMT 100nF 10V 0402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, lib:C0402, F.Cu at (124.5, 62.3)
- added C24: Multilayer Ceramic Capacitors MLCC - SMD/SMT 1uF 6.3V 0402 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, lib:C0402, F.Cu at (125.5, 62.3)
- added C3: Multilayer Ceramic Capacitors MLCC - SMD/SMT 10uF 10V 0805 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, lib:C0805, F.Cu at (134.0, 53.4)
- added C4: Multilayer Ceramic Capacitors MLCC - SMD/SMT 10uF 10V 0805 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, lib:C0805, F.Cu at (134.0, 55.4)
- added C5: Multilayer Ceramic Capacitors MLCC - SMD/SMT 100nF 10V 0402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, lib:C0402, F.Cu at (131.2, 50.8)
- added C6: Multilayer Ceramic Capacitors MLCC - SMD/SMT 10uF 10V 0805 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, lib:C0805, F.Cu at (144.5, 54.4)
- added C7: Multilayer Ceramic Capacitors MLCC - SMD/SMT 10uF 10V 0805 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, lib:C0805, F.Cu at (144.5, 52.4)
- added C8: Multilayer Ceramic Capacitors MLCC - SMD/SMT 10uF 10V 0805 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, lib:C0805, F.Cu at (144.3, 61.6)
- added C9: Multilayer Ceramic Capacitors MLCC - SMD/SMT 10uF 10V 0805 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, lib:C0805, F.Cu at (144.3, 63.6)
- added L1: , lib:IND-SMD_L2.5-W2.0_WPN252012H, F.Cu at (138.3, 49.4)
- added L2: , lib:IND-SMD_L2.5-W2.0_WPN252012H, F.Cu at (148.7, 57.7)
- added LED1: , lib:LED0603-RD, F.Cu at (142.0, 41.6)
- added LED2: , lib:LED0603-RD, F.Cu at (145.0, 41.6)
- added R1: Chip Resistor - Surface Mount 1MOhms ±5% 1/16W 0402 RoHS, lib:R0402, F.Cu at (134.7, 51.9)
- added R10: Chip Resistor - Surface Mount 120Ohms ±5% 1/16W 0402 RoHS, lib:R0402, F.Cu at (141.0, 43.4)
- added R11: Chip Resistor - Surface Mount 82Ohms ±5% 1/16W 0402 RoHS, lib:R0402, F.Cu at (145.8, 43.5)
- added R12: Chip Resistor - Surface Mount 1KOhms ±5% 1/16W 0402 RoHS, lib:R0402, F.Cu at (122.0, 61.2)
- added R13: Chip Resistor - Surface Mount 27KOhms ±5% 1/16W 0402 RoHS, lib:R0402, F.Cu at (125.9, 49.3)
- added R14: Chip Resistor - Surface Mount 27KOhms ±5% 1/16W 0402 RoHS, lib:R0402, F.Cu at (125.9, 50.4)
- added R15: Chip Resistor - Surface Mount 11KOhms ±5% 1/16W 0402 RoHS, lib:R0402, F.Cu at (116.8, 56.3)
- added R16: Chip Resistor - Surface Mount 10KOhms ±5% 1/16W 0402 RoHS, lib:R0402, F.Cu at (118.9, 50.4)
- added R2: Chip Resistor - Surface Mount 180KOhms ±5% 1/16W 0402 RoHS, lib:R0402, F.Cu at (132.8, 51.9)
- added R3: Chip Resistor - Surface Mount 1MOhms ±5% 1/16W 0402 RoHS, lib:R0402, F.Cu at (131.3, 47.8)
- added R4: Chip Resistor - Surface Mount 1.6MOhms ±5% 1/16W 0402 RoHS, lib:R0402, F.Cu at (145.1, 60.1)
- added R5: Chip Resistor - Surface Mount 180KOhms ±5% 1/16W 0402 RoHS, lib:R0402, F.Cu at (143.2, 60.1)
- added R6: Chip Resistor - Surface Mount 1MOhms ±5% 1/16W 0402 RoHS, lib:R0402, F.Cu at (141.6, 56.1)
- added R7: Chip Resistor - Surface Mount 4.7KOhms ±5% 1/16W 0402 RoHS, lib:R0402, F.Cu at (133.5, 60.7)
- added R8: Chip Resistor - Surface Mount 4.7KOhms ±5% 1/16W 0402 RoHS, lib:R0402, F.Cu at (136.5, 60.7)
- added R9: Chip Resistor - Surface Mount 560Ohms ±5% 1/16W 0402 RoHS, lib:R0402, F.Cu at (142.5, 42.9)
- added U1: , Connector_PinHeader_1.27mm:PinHeader_1x02_P1.27mm_Vertical, F.Cu at (134.6, 41.1)
- added U10: , lib:LED-SMD_4P-L2.0-W2.0-BR, F.Cu at (55.9, 122.4)
- added U11: , lib:LED-SMD_4P-L2.0-W2.0-BR, F.Cu at (58.9, 122.4)
- added U12: , lib:LED-SMD_4P-L2.0-W2.0-BR, F.Cu at (62.0, 122.4)
- added U13: , lib:LED-SMD_4P-L2.0-W2.0-BR, F.Cu at (65.0, 122.4)
- added U14: , lib:LED-SMD_4P-L2.0-W2.0-BR, F.Cu at (68.1, 122.4)
- added U15: , lib:LED-SMD_4P-L2.0-W2.0-BR, F.Cu at (71.1, 122.4)
- added U16: , lib:LED-SMD_4P-L2.0-W2.0-BR, F.Cu at (74.2, 122.4)
- added U17: , lib:LED-SMD_4P-L2.0-W2.0-BR, F.Cu at (77.2, 122.4)
- added U18: , lib:LED-SMD_4P-L2.0-W2.0-BR, F.Cu at (-85.2, 202.3)
- added U19: , lib:LED-SMD_4P-L2.0-W2.0-BR, F.Cu at (-51.2, 261.8)
- added U2: , lib:VSON-14_L4.0-W3.0-P0.50-BL-EP_TI_DSJ, F.Cu at (134.5, 49.3)
- added U20: , lib:LED-SMD_4P-L2.0-W2.0-BR, F.Cu at (-110.7, 202.3)
- added U21: , lib:LED-SMD_4P-L2.0-W2.0-BR, F.Cu at (-59.7, 219.3)
- added U22: , lib:LED-SMD_4P-L2.0-W2.0-BR, F.Cu at (-102.2, 185.3)
- added U23: , lib:LED-SMD_4P-L2.0-W2.0-BR, F.Cu at (-127.7, 236.3)
- added U24: , lib:LED-SMD_4P-L2.0-W2.0-BR, F.Cu at (-119.2, 278.8)
- added U25: , lib:LED-SMD_4P-L2.0-W2.0-BR, F.Cu at (-93.7, 219.3)
- added U26: , lib:LED-SMD_4P-L2.0-W2.0-BR, F.Cu at (-153.2, 270.3)
- added U27: , lib:LED-SMD_4P-L2.0-W2.0-BR, F.Cu at (-68.2, 219.3)
- added U28: , lib:LED-SMD_4P-L2.0-W2.0-BR, F.Cu at (-59.7, 261.8)
- added U29: , lib:LED-SMD_4P-L2.0-W2.0-BR, F.Cu at (-153.2, 168.3)
- added U3: , lib:VSON-14_L4.0-W3.0-P0.50-BL-EP_TI_DSJ, F.Cu at (144.9, 57.5)
- added U30: , lib:LED-SMD_4P-L2.0-W2.0-BR, F.Cu at (-119.2, 168.3)
- added U31: , lib:LED-SMD_4P-L2.0-W2.0-BR, F.Cu at (-110.7, 261.8)
- added U32: , lib:LED-SMD_4P-L2.0-W2.0-BR, F.Cu at (-170.2, 159.8)
- added U33: , lib:LED-SMD_4P-L2.0-W2.0-BR, F.Cu at (-170.2, 278.8)
- added U34: , lib:LED-SMD_4P-L2.0-W2.0-BR, F.Cu at (-68.2, 236.3)
- added U35: , lib:LED-SMD_4P-L2.0-W2.0-BR, F.Cu at (-161.7, 227.8)
- added U36: , lib:LED-SMD_4P-L2.0-W2.0-BR, F.Cu at (-76.7, 210.8)
- added U37: , lib:LED-SMD_4P-L2.0-W2.0-BR, F.Cu at (-170.2, 193.8)
- added U38: , lib:LED-SMD_4P-L2.0-W2.0-BR, F.Cu at (-127.7, 176.8)
- added U39: , lib:LED-SMD_4P-L2.0-W2.0-BR, F.Cu at (-76.7, 168.3)
- added U4: , lib:USB-C-SMD_KH-TYPE-C-16P, F.Cu at (134.7, 65.2)
- added U40: , lib:LED-SMD_4P-L2.0-W2.0-BR, F.Cu at (-119.2, 185.3)
- added U41: , lib:LED-SMD_4P-L2.0-W2.0-BR, F.Cu at (-85.2, 168.3)
- added U42: , lib:LED-SMD_4P-L2.0-W2.0-BR, F.Cu at (-144.7, 151.3)
- added U43: , lib:LED-SMD_4P-L2.0-W2.0-BR, F.Cu at (-110.7, 185.3)
- added U44: , lib:LED-SMD_4P-L2.0-W2.0-BR, F.Cu at (-51.2, 202.3)
- added U45: , lib:LED-SMD_4P-L2.0-W2.0-BR, F.Cu at (-153.2, 253.3)
- added U46: , lib:LED-SMD_4P-L2.0-W2.0-BR, F.Cu at (-93.7, 176.8)
- added U47: , lib:LED-SMD_4P-L2.0-W2.0-BR, F.Cu at (-178.7, 193.8)
- added U48: , lib:LED-SMD_4P-L2.0-W2.0-BR, F.Cu at (-161.7, 210.8)
- added U49: , lib:LED-SMD_4P-L2.0-W2.0-BR, F.Cu at (-76.7, 227.8)
- added U5: , lib:WSON-10_L2.0-W2.0-P0.40-BL-EP, F.Cu at (143.6, 44.7)
- added U50: , lib:LED-SMD_4P-L2.0-W2.0-BR, F.Cu at (-51.2, 278.8)
- added U51: , lib:LED-SMD_4P-L2.0-W2.0-BR, F.Cu at (-119.2, 270.3)
- added U52: , lib:LED-SMD_4P-L2.0-W2.0-BR, F.Cu at (-136.2, 159.8)
- added U53: , lib:LED-SMD_4P-L2.0-W2.0-BR, F.Cu at (-76.7, 176.8)
- added U54: , lib:LED-SMD_4P-L2.0-W2.0-BR, F.Cu at (-170.2, 227.8)
- added U55: , lib:LED-SMD_4P-L2.0-W2.0-BR, F.Cu at (-178.7, 261.8)
- added U56: , lib:LED-SMD_4P-L2.0-W2.0-BR, F.Cu at (-161.7, 151.3)
- added U57: , lib:LED-SMD_4P-L2.0-W2.0-BR, F.Cu at (-161.7, 168.3)
- added U58: , lib:LED-SMD_4P-L2.0-W2.0-BR, F.Cu at (-136.2, 219.3)
- added U59: , lib:LED-SMD_4P-L2.0-W2.0-BR, F.Cu at (-178.7, 270.3)
- added U6: , lib:LQFN-56_L7.0-W7.0-P0.4-EP, F.Cu at (122.1, 55.2)
- added U60: , lib:LED-SMD_4P-L2.0-W2.0-BR, F.Cu at (-119.2, 210.8)
- added U61: , lib:LED-SMD_4P-L2.0-W2.0-BR, F.Cu at (-85.2, 219.3)
- added U62: , lib:LED-SMD_4P-L2.0-W2.0-BR, F.Cu at (-127.7, 151.3)
- added U63: , lib:LED-SMD_4P-L2.0-W2.0-BR, F.Cu at (-127.7, 253.3)
- added U64: , lib:LED-SMD_4P-L2.0-W2.0-BR, F.Cu at (-153.2, 244.8)
- added U65: , lib:LED-SMD_4P-L2.0-W2.0-BR, F.Cu at (-110.7, 244.8)
- added U66: , lib:LED-SMD_4P-L2.0-W2.0-BR, F.Cu at (-51.2, 168.3)
- added U67: , lib:LED-SMD_4P-L2.0-W2.0-BR, F.Cu at (-68.2, 227.8)
- added U68: , lib:LED-SMD_4P-L2.0-W2.0-BR, F.Cu at (-110.7, 168.3)
- added U69: , lib:LED-SMD_4P-L2.0-W2.0-BR, F.Cu at (-119.2, 219.3)
- added U7: , lib:OSC-SMD_4P-L3.2-W2.5-BL, F.Cu at (120.8, 63.5)
- added U70: , lib:LED-SMD_4P-L2.0-W2.0-BR, F.Cu at (-127.7, 193.8)
- added U71: , lib:LED-SMD_4P-L2.0-W2.0-BR, F.Cu at (-51.2, 185.3)
- added U72: , lib:LED-SMD_4P-L2.0-W2.0-BR, F.Cu at (-127.7, 210.8)
- added U73: , lib:LED-SMD_4P-L2.0-W2.0-BR, F.Cu at (-59.7, 227.8)
- added U74: , lib:LED-SMD_4P-L2.0-W2.0-BR, F.Cu at (-93.7, 151.3)
- added U75: , lib:LED-SMD_4P-L2.0-W2.0-BR, F.Cu at (-136.2, 202.3)
- added U76: , lib:LED-SMD_4P-L2.0-W2.0-BR, F.Cu at (-51.2, 151.3)
- added U77: , lib:LED-SMD_4P-L2.0-W2.0-BR, F.Cu at (-144.7, 210.8)
- added U78: , lib:LED-SMD_4P-L2.0-W2.0-BR, F.Cu at (-153.2, 278.8)
- added U79: , lib:LED-SMD_4P-L2.0-W2.0-BR, F.Cu at (-76.7, 270.3)
- added U8: , lib:SOIC-8_L5.3-W5.3-P1.27-LS8.0-BL, F.Cu at (122.2, 46.3)
- added U80: , lib:LED-SMD_4P-L2.0-W2.0-BR, F.Cu at (-110.7, 236.3)
- added U81: , lib:LED-SMD_4P-L2.0-W2.0-BR, F.Cu at (-59.7, 244.8)
- added U82: , lib:LED-SMD_4P-L2.0-W2.0-BR, F.Cu at (-144.7, 219.3)
- added U83: , lib:LED-SMD_4P-L2.0-W2.0-BR, F.Cu at (-52.5, 140.0)
- added U84: , lib:LED-SMD_4P-L2.0-W2.0-BR, F.Cu at (-102.2, 227.8)
- added U85: , lib:LED-SMD_4P-L2.0-W2.0-BR, F.Cu at (-144.7, 227.8)
- added U86: , lib:LED-SMD_4P-L2.0-W2.0-BR, F.Cu at (-127.7, 168.3)
- added U87: , lib:LED-SMD_4P-L2.0-W2.0-BR, F.Cu at (-110.7, 219.3)
- added U88: , lib:LED-SMD_4P-L2.0-W2.0-BR, F.Cu at (-68.2, 176.8)
- added U89: , lib:LED-SMD_4P-L2.0-W2.0-BR, F.Cu at (-85.2, 185.3)
- added U9: , lib:LED-SMD_4P-L2.0-W2.0-BR, F.Cu at (52.8, 122.4)
- added U90: , lib:LED-SMD_4P-L2.0-W2.0-BR, F.Cu at (-78.0, 140.0)
- added U91: , lib:LED-SMD_4P-L2.0-W2.0-BR, F.Cu at (-178.7, 236.3)
- added U92: , lib:LED-SMD_4P-L2.0-W2.0-BR, F.Cu at (-110.7, 210.8)
- added U93: , lib:LED-SMD_4P-L2.0-W2.0-BR, F.Cu at (-178.7, 210.8)
- added U94: , lib:LED-SMD_4P-L2.0-W2.0-BR, F.Cu at (-76.7, 278.8)
- added U95: , lib:LED-SMD_4P-L2.0-W2.0-BR, F.Cu at (-102.2, 253.3)
- added U96: , lib:LED-SMD_4P-L2.0-W2.0-BR, F.Cu at (-51.2, 227.8)
- added U97: , lib:LED-SMD_4P-L2.0-W2.0-BR, F.Cu at (-85.2, 227.8)
- added U98: , lib:LED-SMD_4P-L2.0-W2.0-BR, F.Cu at (-93.7, 227.8)
Routing:
- net vcc-1: track 0.00 -> 48.7 mm, vias 0 -> 3
- net vcc-6: track 0.00 -> 23.4 mm, vias 0 -> 2
- net vcc: track 0.00 -> 15.4 mm
- net sck: track 0.00 -> 14.4 mm
- net gnd: track 0.00 -> 13.9 mm, vias 0 -> 2
- net io0: track 0.00 -> 12.8 mm, vias 0 -> 2
- net io3: track 0.00 -> 9.73 mm
- net io1: track 0.00 -> 9.57 mm
- net cs: track 0.00 -> 9.55 mm
- net xin: track 0.00 -> 8.08 mm
- net io2: track 0.00 -> 6.20 mm
- net vcc-2: track 0.00 -> 6.20 mm
- net vcc-3: track 0.00 -> 6.03 mm, vias 0 -> 2
- net usb_dp: track 0.00 -> 4.15 mm
- net out-2: track 0.00 -> 3.72 mm
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Other:
- board size 225.7 x 100.8 mm -> 40 x 40 mm
